Commit message: urdf file

File: urdf/fire_truck.urdf (robot description, URDF)
Before this commit: robot firetruck_robot, 7 links, 6 joints
Joints:
- joint front_wheel_joint: limit (none) -> effort=100 velocity=20
- joint left_wheel_joint: limit (none) -> effort=100 velocity=20
- joint right_wheel_joint: limit (none) -> effort=100 velocity=20
- joint rotation_joint: limit (none) -> effort=100 velocity=20

Commit message: urdf file met betere extension

File: urdf/fire_truck.urdf (robot description, URDF)
Before this commit: robot firetruck_robot, 7 links, 6 joints
Links:
- link front_wheel: geometry collision cylinder length=0.06 radius=0.15; visual cylinder length=0.06 radius=0.15
- link left_wheel: geometry collision cylinder length=0.06 radius=0.15; visual cylinder length=0.06 radius=0.15
- link right_wheel: geometry collision cylinder length=0.06 radius=0.15; visual cylinder length=0.06 radius=0.15
Joints:
- joint extend_joint: limit lower=0 upper=0.5 effort=50 velocity=1.0 -> lower=0 upper=2 effort=50 velocity=1.0; origin xyz=0.25 0 0.05 rpy=0 0 0 -> xyz=0.25 0 0 rpy=0 0 0
- joint left_wheel_joint: origin xyz=-0.3 -0.4 0 rpy=0 0 0 -> xyz=-0.28 -0.4 0 rpy=0 0 0
- joint right_wheel_joint: origin xyz=-0.3 0.4 0 rpy=0 0 0 -> xyz=-0.28 0.4 0 rpy=0 0 0

Commit message: voorste wiel can nu draaien

File: urdf/fire_truck.urdf (robot description, URDF)
Before this commit: robot firetruck_robot, 7 links, 6 joints
Joints:
- joint front_wheel_joint: axis 0 1 0 -> 0 1 1

Commit message: final repository

File: urdf/fire_truck.urdf (robot description, URDF)
Before this commit: robot firetruck_robot, 7 links, 6 joints
Joints:
- joint left_wheel_joint: origin xyz=-0.28 -0.4 0 rpy=0 0 0 -> xyz=-0.28 -0.2 0 rpy=0 0 0
- joint right_wheel_joint: origin xyz=-0.28 0.4 0 rpy=0 0 0 -> xyz=-0.28 0.2 0 rpy=0 0 0
